File: LoRa_thing/LoRa_thing.kicad_pcb (KiCad board)
At the start: 2 copper layers, 47.6 x 73.7 mm, 3 parts, among them U1 Ai-Thinker-Ra-02, U2 Pico

Commit message: un peu de travail
Parts:
- added J1: 3V3, Connector_PinHeader_2.54mm:PinHeader_1x01_P2.54mm_Vertical, F.Cu at (134.6, 104.1)
Routing:
- net Net-(B1-Pad2): track 96.8 -> 99.1 mm
Other:
- board size 47.6 x 73.7 mm -> 43.2 x 73.7 mm
