File: LoRa_thing/LoRa_thing.kicad_sch (KiCad schematic)
At the start: 3 parts, among them U1 Ai-Thinker-Ra-02, U2 Pico

Commit message: un peu de travail
Parts:
- added J1: 3V3, Connector_PinHeader_2.54mm:PinHeader_1x01_P2.54mm_Vertical, symbol Connector:Conn_01x01_Male
Connections:
- net at B1.2 (3v3), U1.3 (VDD), U2.36 (3V3): now also J1.1 (Pin_1)
Changed lines of the file:
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@@
 (kicad_sch (version 20211123) (generator eeschema)
   (paper "A4")
+  (junction (at 189.23 46.99) (diameter 0) (color 0 0 0 0)
+  )
   (junction (at 187.96 83.82) (diameter 0) (color 0 0 0 0)
   )
@@
     (stroke (width 0) (type default) (color 0 0 0 0))
   )
+  (wire (pts (xy 189.23 46.99) (xy 191.77 46.99))
+    (stroke (width 0) (type default) (color 0 0 0 0))
+  )
   (wire (pts (xy 189.23 88.9) (xy 182.88 88.9))
     (stroke (width 0) (type default) (color 0 0 0 0))
@@
     (stroke (width 0) (type default) (color 0 0 0 0))
   )
+  (wire (pts (xy 189.23 46.99) (xy 189.23 71.12))
+    (stroke (width 0) (type default) (color 0 0 0 0))
+  )
   (wire (pts (xy 124.46 109.22) (xy 147.32 109.22))
     (stroke (width 0) (type default) (color 0 0 0 0))
@@
     (stroke (width 0) (type default) (color 0 0 0 0))
   )
-  (wire (pts (xy 189.23 34.29) (xy 189.23 71.12))
+  (wire (pts (xy 189.23 34.29) (xy 189.23 46.99))
     (stroke (width 0) (type default) (color 0 0 0 0))
   )
@@
     (pin "8")
     (pin "9")
+  )
+  (symbol (lib_id "Connector:Conn_01x01_Male") (at 196.85 46.99 0) (mirror y) (unit 1)
+    (in_bom yes) (on_board yes) (fields_autoplaced)
+    (property "Reference" "J1" (id 0) (at 196.215 41.91 0))
+    (property "Value" "3V3" (id 1) (at 196.215 44.45 0))
+    (property "Footprint" "Connector_PinHeader_2.54mm:PinHeader_1x01_P2.54mm_Vertical" (id 2) (at 196.85 46.99 0)
+      (effects (font (size 1.27 1.27)) hide)
+    )
+    (property "Datasheet" "~" (id 3) (at 196.85 46.99 0)
+      (effects (font (size 1.27 1.27)) hide)
+    )
+    (pin "1")
   )
   (symbol (lib_id "power:GND") (at 139.7 125.73 0) (unit 1)
@@
       (reference "B1") (unit 1) (value "AdafruitThinkInk") (footprint "Library:Adafruit ThinkInk Tricolor 200")
     )
+    (path "/e294d04e-3720-4cda-b63e-078484e0733c"
+      (reference "J1") (unit 1) (value "3V3") (footprint "Connector_PinHeader_2.54mm:PinHeader_1x01_P2.54mm_Vertical")
+    )
     (path "/ce23a379-659a-440d-9e9b-17e56c093d24"
