File: Pi_Keyboard/Pi_Keyboard.kicad_pcb (KiCad board)
At the start: 2 copper layers, 43.2 x 35.6 mm, 69 parts, among them SW1 SW_Push, SW10 SW_Push, SW11 SW_Push, SW12 SW_Push, SW13 SW_Push, SW14 SW_Push, SW15 SW_Push, SW16 SW_Push, SW17 SW_Push, SW18 SW_Push, SW19 SW_Push, SW2 SW_Push, SW20 SW_Push, SW21 SW_Push, SW22 SW_Push, SW23 SW_Push, SW24 SW_Push, SW25 SW_Push, SW26 SW_Push, SW27 SW_Push, SW28 SW_Push, SW29 SW_Push, SW3 SW_Push, SW30 SW_Push, SW31 SW_Push, SW32 SW_Push, SW4 SW_Push, SW5 SW_Push, SW6 SW_Push, SW7 SW_Push, SW8 SW_Push, SW9 SW_Push, U1 74HC165, U2 74HC165, U3 Pico, U4 74HC165, U5 74HC165

Commit message: un peu de travail
Parts:
- added 3V3: Conn_01x01_Male, Library:PinHeader_1x01_P2.54mm_Vertical, F.Cu at (125.1, 91.4)
- A1: renamed from SW8; value SW_Push -> ^
- D1: renamed from SW6; value SW_Push -> S
- E1: renamed from SW3; value SW_Push -> E
- F1: renamed from SW5; value SW_Push -> D
- Q1: renamed from SW1; value SW_Push -> Q
- R1, R10, R11, R12, R13, R14, R15, R16, R17, R18, R19, R2, R20, R21, R22, R23, R24, R25, R26, R27, R28, R29, R3, R30, R31, R32, R4, R5, R6, R7, R8, R9: footprint Resistor_SMD:R_0603_1608Metric -> Library:R_0603_1608Metric
- R33: renamed from SW4; value SW_Push -> R
- S1: renamed from SW7; value SW_Push -> A
- SW10: value SW_Push -> Z
- SW11: value SW_Push -> X
- SW12: value SW_Push -> C
- SW13: value SW_Push -> V
- SW14: value SW_Push -> F
- SW15: value SW_Push -> T
- SW16: value SW_Push -> Y
- SW17: value SW_Push -> G
- SW18: value SW_Push -> U
- SW19: value SW_Push -> H
- SW20: value SW_Push -> B
- SW21: value SW_Push -> N
- SW22: value SW_Push -> M
- SW23: value SW_Push -> _
- SW24: value SW_Push -> #
- SW25: value SW_Push -> ^^
- SW26: value SW_Push -> L
- SW27: value SW_Push -> K
- SW28: value SW_Push -> J
- SW29: value SW_Push -> I
- SW30: value SW_Push -> O
- SW31: value SW_Push -> P
- SW32: value SW_Push -> *
- SW9: value SW_Push -> $
- U1, U2, U4, U5: footprint Package_SO:SOIC-16_3.9x9.9mm_P1.27mm -> Library:SOIC-16_3.9x9.9mm_P1.27mm
- U3: footprint MCU_RaspberryPi_and_Boards:RPi_Pico_Pin_ -> Library:RPi_Pico_Pin_
- W1: renamed from SW2; value SW_Push -> W
- moved R32 48.3 mm to (130.3, 121.3), turned to 90 degrees
- moved R23 47.9 mm to (125.7, 118.7), turned to 180 degrees
- moved R17 42.3 mm to (113.0, 111.1), turned to 180 degrees
- moved R18 41.3 mm to (116.8, 103.5), turned to 180 degrees
- moved R24 40.9 mm to (131.0, 124.5), turned to 180 degrees
- moved R20 40.8 mm to (114.3, 118.7), turned to 180 degrees
- moved R29 40.6 mm to (120.7, 103.6), turned to 180 degrees
- moved R19 40.3 mm to (116.8, 111.1), turned to 180 degrees
- moved R22 40.2 mm to (121.9, 118.7), turned to 180 degrees
- moved R27 37.3 mm to (124.5, 111.1), turned to 180 degrees
- moved R15 35.5 mm to (109.2, 103.5), turned to 180 degrees
- moved R25 35.0 mm to (131.8, 121.3), turned to 90 degrees
- moved R16 33.4 mm to (113.0, 103.5), turned to 180 degrees
- moved R28 32.3 mm to (120.7, 111.1), turned to 180 degrees
- moved R30 30.6 mm to (124.5, 103.6), turned to 180 degrees
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Connections:
- R1 pad 1: Net-(R1-Pad1) -> Net-(R25-Pad1)
- R10 pad 1: Net-(R10-Pad1) -> Net-(R25-Pad1)
- R11 pad 1: Net-(R10-Pad1) -> Net-(R25-Pad1)
- R12 pad 1: Net-(R10-Pad1) -> Net-(R25-Pad1)
- R13 pad 1: Net-(R10-Pad1) -> Net-(R25-Pad1)
- R14 pad 1: Net-(R10-Pad1) -> Net-(R25-Pad1)
- R15 pad 1: Net-(R10-Pad1) -> Net-(R25-Pad1)
- R16 pad 1: Net-(R10-Pad1) -> Net-(R25-Pad1)
- R17 pad 1: Net-(R17-Pad1) -> Net-(R25-Pad1)
- R18 pad 1: Net-(R17-Pad1) -> Net-(R25-Pad1)
- R19 pad 1: Net-(R17-Pad1) -> Net-(R25-Pad1)
- R2 pad 1: Net-(R1-Pad1) -> Net-(R25-Pad1)
- R20 pad 1: Net-(R17-Pad1) -> Net-(R25-Pad1)
- R21 pad 1: Net-(R17-Pad1) -> Net-(R25-Pad1)
- R22 pad 1: Net-(R17-Pad1) -> Net-(R25-Pad1)
- R23 pad 1: Net-(R17-Pad1) -> Net-(R25-Pad1)
- R24 pad 1: Net-(R17-Pad1) -> Net-(R25-Pad1)
- R3 pad 1: Net-(R1-Pad1) -> Net-(R25-Pad1)
- R4 pad 1: Net-(R1-Pad1) -> Net-(R25-Pad1)
- R5 pad 1: Net-(R1-Pad1) -> Net-(R25-Pad1)
- R6 pad 1: Net-(R1-Pad1) -> Net-(R25-Pad1)
- R7 pad 1: Net-(R1-Pad1) -> Net-(R25-Pad1)
- R8 pad 1: Net-(R1-Pad1) -> Net-(R25-Pad1)
- R9 pad 1: Net-(R10-Pad1) -> Net-(R25-Pad1)
- U3 pad 19: unconnected-(U3-Pad19) -> PL
- U3 pad 20: unconnected-(U3-Pad20) -> CP
- U3 pad 21: unconnected-(U3-Pad21) -> Net-(U3-Pad21)
- U3 pad 22: unconnected-(U3-Pad22) -> Net-(R25-Pad1)
- U3 pad 36: +3V3 -> unconnected-(U3-Pad36)
- U5 pad 9: unconnected-(U5-Pad9) -> Net-(U3-Pad21)
Routing:
- net Net-(R25-Pad1): track 0.00 -> 248.7 mm, vias 0 -> 14
- net Net-(SW24-Pad2): track 0.00 -> 41.0 mm, vias 0 -> 2
- net Net-(SW23-Pad2): track 0.00 -> 36.3 mm, vias 0 -> 2
- net CP: track 8.15 -> 42.8 mm
- net Net-(R1-Pad1): track 32.7 -> 0.00 mm
- net Net-(SW22-Pad2): track 0.00 -> 32.0 mm, vias 0 -> 2
- net Net-(SW20-Pad2): track 0.00 -> 29.9 mm, vias 0 -> 2
- net Net-(SW13-Pad2): track 0.00 -> 29.7 mm, vias 0 -> 2
- net Net-(SW21-Pad2): track 0.00 -> 28.8 mm, vias 0 -> 2
- net Net-(SW27-Pad2): track 0.00 -> 26.5 mm, vias 0 -> 2
- net Net-(SW17-Pad2): track 0.00 -> 26.5 mm, vias 0 -> 2
- net Net-(SW28-Pad2): track 0.00 -> 26.2 mm, vias 0 -> 2
- net PL: track 0.07 -> 25.9 mm
- net Net-(SW19-Pad2): track 0.00 -> 23.7 mm, vias 0 -> 2
- net Net-(SW26-Pad2): track 0.00 -> 23.0 mm, vias 0 -> 2
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
Commit message: some
Parts:
- 3V3: footprint Library:PinHeader_1x01_P2.54mm_Vertical -> Connector_PinHeader_2.54mm:PinHeader_1x01_P2.54mm_Vertical
- R1, R10, R11, R12, R13, R14, R15, R16, R17, R18, R19, R2, R20, R21, R22, R23, R24, R25, R26, R27, R28, R29, R3, R30, R31, R32, R4, R5, R6, R7, R8, R9: footprint Library:R_0603_1608Metric -> Resistor_SMD:R_0603_1608Metric
- U3: footprint Library:RPi_Pico_Pin_ -> MCU_RaspberryPi_and_Boards:RPi_Pico_Pin_
- moved R10 105.3 mm to (23.3, 45.6)
- moved R11 105.3 mm to (27.1, 45.6)
- moved R12 105.3 mm to (30.9, 45.6)
- moved R13 105.3 mm to (34.7, 45.6)
- moved R20 105.3 mm to (38.5, 45.6)
- moved R21 105.3 mm to (42.3, 45.6)
- moved R22 105.3 mm to (46.1, 45.6)
- moved R23 105.3 mm to (49.9, 45.6)
- moved R9 105.3 mm to (19.5, 45.6)
- moved SW10 105.3 mm to (21.4, 49.4)
- moved SW11 105.3 mm to (25.2, 49.4)
- moved SW12 105.3 mm to (29.0, 49.4)
- moved SW13 105.3 mm to (32.8, 49.4)
- moved SW20 105.3 mm to (36.6, 49.4)
- moved SW21 105.3 mm to (40.4, 49.4)
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- renumbered Q1 to SW1, W1 to SW2, E1 to SW3, R33 to SW4, F1 to SW5, D1 to SW6, S1 to SW7, A1 to SW8
Connections:
- net Net-(R25-Pad1) renamed PULL
- SW1 pad 2: Net-(Q1-Pad2) -> SET
- SW10 pad 2: Net-(SW10-Pad2) -> SET
- SW11 pad 2: Net-(SW11-Pad2) -> SET
- SW12 pad 2: Net-(SW12-Pad2) -> SET
- SW13 pad 2: Net-(SW13-Pad2) -> SET
- SW14 pad 2: Net-(SW14-Pad2) -> SET
- SW15 pad 2: Net-(SW15-Pad2) -> SET
- SW16 pad 2: Net-(SW16-Pad2) -> SET
- SW17 pad 2: Net-(SW17-Pad2) -> SET
- SW18 pad 2: Net-(SW18-Pad2) -> SET
- SW19 pad 2: Net-(SW19-Pad2) -> SET
- SW2 pad 2: Net-(W1-Pad2) -> SET
- SW20 pad 2: Net-(SW20-Pad2) -> SET
- SW21 pad 2: Net-(SW21-Pad2) -> SET
- SW22 pad 2: Net-(SW22-Pad2) -> SET
- SW23 pad 2: Net-(SW23-Pad2) -> SET
- SW24 pad 2: Net-(SW24-Pad2) -> SET
- SW25 pad 2: Net-(SW25-Pad2) -> SET
- SW26 pad 2: Net-(SW26-Pad2) -> SET
- SW27 pad 2: Net-(SW27-Pad2) -> SET
- SW28 pad 2: Net-(SW28-Pad2) -> SET
- SW29 pad 2: Net-(SW29-Pad2) -> SET
- SW3 pad 2: Net-(E1-Pad2) -> SET
- SW30 pad 2: Net-(SW30-Pad2) -> SET
- SW31 pad 2: Net-(SW31-Pad2) -> SET
- SW32 pad 2: Net-(SW32-Pad2) -> SET
- SW4 pad 2: Net-(R33-Pad2) -> SET
- SW5 pad 2: Net-(F1-Pad2) -> SET
- SW6 pad 2: Net-(D1-Pad2) -> SET
- SW7 pad 2: Net-(S1-Pad2) -> SET
- SW8 pad 2: Net-(A1-Pad2) -> SET
- SW9 pad 2: Net-(SW9-Pad2) -> SET
- U1 pad 10: GND -> SET
- U1 pad 11: Net-(Q1-Pad2) -> Net-(R1-Pad2)
- U1 pad 12: Net-(W1-Pad2) -> Net-(R2-Pad2)
- U1 pad 13: Net-(E1-Pad2) -> Net-(R3-Pad2)
- U1 pad 14: Net-(R33-Pad2) -> Net-(R4-Pad2)
- U1 pad 15: GND -> SET
- U1 pad 3: Net-(F1-Pad2) -> Net-(R5-Pad2)
- U1 pad 4: Net-(D1-Pad2) -> Net-(R6-Pad2)
- U1 pad 5: Net-(S1-Pad2) -> Net-(R7-Pad2)
- U1 pad 6: Net-(A1-Pad2) -> Net-(R8-Pad2)
- U1 pad 8: GND -> SET
- U2 pad 11: Net-(SW9-Pad2) -> Net-(R9-Pad2)
- U2 pad 12: Net-(SW10-Pad2) -> Net-(R10-Pad2)
- U2 pad 13: Net-(SW11-Pad2) -> Net-(R11-Pad2)
- U2 pad 14: Net-(SW12-Pad2) -> Net-(R12-Pad2)
- U2 pad 15: GND -> SET
- U2 pad 3: Net-(SW13-Pad2) -> Net-(R13-Pad2)
- U2 pad 4: Net-(SW14-Pad2) -> Net-(R14-Pad2)
- U2 pad 5: Net-(SW15-Pad2) -> Net-(R15-Pad2)
- U2 pad 6: Net-(SW16-Pad2) -> Net-(R16-Pad2)
- U2 pad 8: GND -> SET
- U3 pad 18: GND -> SET
- U3 pad 23: GND -> SET
- U4 pad 11: Net-(SW17-Pad2) -> Net-(R17-Pad2)
- U4 pad 12: Net-(SW18-Pad2) -> Net-(R18-Pad2)
- U4 pad 13: Net-(SW19-Pad2) -> Net-(R19-Pad2)
- U4 pad 14: Net-(SW20-Pad2) -> Net-(R20-Pad2)
- U4 pad 15: GND -> SET
- U4 pad 3: Net-(SW21-Pad2) -> Net-(R21-Pad2)
- U4 pad 4: Net-(SW22-Pad2) -> Net-(R22-Pad2)
- U4 pad 5: Net-(SW23-Pad2) -> Net-(R23-Pad2)
- U4 pad 6: Net-(SW24-Pad2) -> Net-(R24-Pad2)
- U4 pad 8: GND -> SET
- U5 pad 11: Net-(SW25-Pad2) -> Net-(R25-Pad2)
- U5 pad 12: Net-(SW26-Pad2) -> Net-(R26-Pad2)
- U5 pad 13: Net-(SW27-Pad2) -> Net-(R27-Pad2)
- U5 pad 14: Net-(SW28-Pad2) -> Net-(R28-Pad2)
- U5 pad 15: GND -> SET
- U5 pad 3: Net-(SW29-Pad2) -> Net-(R29-Pad2)
- U5 pad 4: Net-(SW30-Pad2) -> Net-(R30-Pad2)
- U5 pad 5: Net-(SW31-Pad2) -> Net-(R31-Pad2)
- U5 pad 6: Net-(SW32-Pad2) -> Net-(R32-Pad2)
- U5 pad 7: unconnected-(U5-Pad7) -> Net-(U3-Pad21)
- U5 pad 8: GND -> SET
- U5 pad 9: Net-(U3-Pad21) -> unconnected-(U5-Pad9)
Routing:
- net SET: track 0.00 -> 385.5 mm, vias 0 -> 18
- net GND: track 89.2 -> 0.00 mm, vias 6 -> 0
- net Net-(SW24-Pad2): track 41.0 -> 0.00 mm, vias 2 -> 0
- net Net-(SW9-Pad2): track 39.4 -> 0.00 mm, vias 2 -> 0
- net Net-(R9-Pad2): track 6.06 -> 42.4 mm, vias 0 -> 2
- net Net-(SW23-Pad2): track 36.3 -> 0.00 mm, vias 2 -> 0
- net Net-(SW10-Pad2): track 35.4 -> 0.00 mm, vias 2 -> 0
- net Net-(R24-Pad2): track 5.92 -> 40.4 mm, vias 0 -> 2
- net Net-(SW11-Pad2): track 32.6 -> 0.00 mm, vias 2 -> 0
- net Net-(R10-Pad2): track 6.06 -> 38.1 mm, vias 0 -> 2
- net Net-(SW22-Pad2): track 32.0 -> 0.00 mm, vias 2 -> 0
- net Net-(R23-Pad2): track 6.06 -> 36.2 mm, vias 0 -> 2
- net Net-(SW20-Pad2): track 29.9 -> 0.00 mm, vias 2 -> 0
- net Net-(SW13-Pad2): track 29.7 -> 0.00 mm, vias 2 -> 0
- net Net-(SW12-Pad2): track 29.3 -> 0.00 mm, vias 2 -> 0
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Other:
- outline, holes or cut-outs redrawn
