File: Pi_Keyboard/Pi_Keyboard.kicad_sch (KiCad schematic)
At the start: 69 parts, among them SW1 SW_Push, SW10 SW_Push, SW11 SW_Push, SW12 SW_Push, SW13 SW_Push, SW14 SW_Push, SW15 SW_Push, SW16 SW_Push, SW17 SW_Push, SW18 SW_Push, SW19 SW_Push, SW2 SW_Push, SW20 SW_Push, SW21 SW_Push, SW22 SW_Push, SW23 SW_Push, SW24 SW_Push, SW25 SW_Push, SW26 SW_Push, SW27 SW_Push, SW28 SW_Push, SW29 SW_Push, SW3 SW_Push, SW30 SW_Push, SW31 SW_Push, SW32 SW_Push, SW4 SW_Push, SW5 SW_Push, SW6 SW_Push, SW7 SW_Push, SW8 SW_Push, SW9 SW_Push, U1 74HC165, U2 74HC165, U3 Pico, U4 74HC165, U5 74HC165

Commit message: un peu de travail
Parts:
- added 3V3: Conn_01x01_Male, Connector_PinHeader_2.54mm:PinHeader_1x01_P2.54mm_Vertical, symbol Connector:Conn_01x01_Male
- A1: renamed from SW8; value SW_Push -> ^
- D1: renamed from SW6; value SW_Push -> S
- E1: renamed from SW3; value SW_Push -> E
- F1: renamed from SW5; value SW_Push -> D
- Q1: renamed from SW1; value SW_Push -> Q
- R33: renamed from SW4; value SW_Push -> R
- S1: renamed from SW7; value SW_Push -> A
- SW10: value SW_Push -> Z
- SW11: value SW_Push -> X
- SW12: value SW_Push -> C
- SW13: value SW_Push -> V
- SW14: value SW_Push -> F
- SW15: value SW_Push -> T
- SW16: value SW_Push -> Y
- SW17: value SW_Push -> G
- SW18: value SW_Push -> U
- SW19: value SW_Push -> H
- SW20: value SW_Push -> B
- SW21: value SW_Push -> N
- SW22: value SW_Push -> M
- SW23: value SW_Push -> _
- SW24: value SW_Push -> #
- SW25: value SW_Push -> ^^
- SW26: value SW_Push -> L
- SW27: value SW_Push -> K
- SW28: value SW_Push -> J
- SW29: value SW_Push -> I
- SW30: value SW_Push -> O
- SW31: value SW_Push -> P
- SW32: value SW_Push -> *
- SW9: value SW_Push -> $
- W1: renamed from SW2; value SW_Push -> W
Connections:
- net +3V3: now also 3V3.1 (Pin_1); no longer U3.36 (3V3)
- net CP: now also U3.20 (GPIO15)
- net PL: now also U3.19 (GPIO14)
- net at R10.1, R11.1, R12.1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: now also R1.1, R17.1, R18.1, R19.1, R2.1, R20.1, R21.1, R22.1, R23.1, R24.1, R25.1, R26.1, R27.1, R28.1, R29.1, R3.1, R30.1, R31.1, R32.1, R4.1, R5.1, R6.1, R7.1, R8.1, U3.22 (GPIO17)
- net at U5.9 (Q7): now also U3.21 (GPIO16)

Commit message: some
Parts:
- SW25: LCSC (none) -> C411883
- U1, U2, U4, U5: footprint Package_SO:SOIC-16_3.9x9.9mm_P1.27mm -> Library:SOIC-16_3.9x9.9mm_P1.27mm
- U3: footprint MCU_RaspberryPi_and_Boards:RPi_Pico_Pin_ -> RPi_Pico:RPi_Pico_SMD_TH
- renumbered Q1 to SW1, W1 to SW2, E1 to SW3, R33 to SW4, F1 to SW5, D1 to SW6, S1 to SW7, A1 to SW8
Connections:
- net GND: now also SW1.2, SW10.2, SW11.2, SW12.2, SW13.2, SW14.2, SW15.2, SW16.2, SW17.2, SW18.2, SW19.2, SW2.2, SW20.2, SW21.2, SW22.2, SW23.2, SW24.2, SW25.2, SW26.2, SW27.2, SW28.2, SW29.2, SW3.2, SW30.2, SW31.2, SW32.2, SW4.2, SW5.2, SW6.2, SW7.2, SW8.2, SW9.2
- net PULL: now reaches R1.1, R10.1, R11.1, R12.1, R13.1, R14.1, R15.1, R16.1, R17.1, R18.1, R19.1, R2.1, R20.1, R21.1, R22.1, R23.1, R24.1, R25.1, R26.1, R27.1, R28.1, R29.1, R3.1, R30.1, R31.1, R32.1, R4.1, R5.1, R6.1, R7.1, R8.1, R9.1, U3.22 (GPIO17)
- net at R12.2, SW12.1: now also U2.14 (D3)
- net at R10.2, SW10.1: now also U2.12 (D1)
- net at R24.2, SW24.1: now also U4.6 (D7)
- net at R18.2, SW18.1: now also U4.12 (D1)
- net at U2.11 (D0): now also R9.2, SW9.1; no longer SW9.2
- net at U2.13 (D2): now also R11.2, SW11.1; no longer SW11.2
- net at U2.3 (D4): now also R13.2, SW13.1; no longer SW13.2
- net at U2.4 (D5): now also R14.2, SW14.1; no longer SW14.2
- net at U2.5 (D6): now also R15.2, SW15.1; no longer SW15.2
- net at U2.6 (D7): now also R16.2, SW16.1; no longer SW16.2
- net at R19.2, SW19.1: now also U4.13 (D2)
- net at R29.2, SW29.1: now also U5.3 (D4)
- net at R5.2, SW5.1: now also U1.3 (D4)
- net at R23.2, SW23.1: now also U4.5 (D6)
- net at R21.2, SW21.1: now also U4.3 (D4)
- net at R1.2, SW1.1: now also U1.11 (D0)
- net at R28.2, SW28.1: now also U5.14 (D3)
- net at R25.2, SW25.1: now also U5.11 (D0)
- net at R2.2, SW2.1: now also U1.12 (D1)
- net at R27.2, SW27.1: now also U5.13 (D2)
- net at R17.2, SW17.1: now also U4.11 (D0)
- net at U1.13 (D2): now also R3.2, SW3.1; no longer SW3.2
- net at U1.14 (D3): now also R4.2, SW4.1; no longer SW4.2
- net at U1.4 (D5): now also R6.2, SW6.1; no longer SW6.2
- net at U1.5 (D6): now also R7.2, SW7.1; no longer SW7.2
- net at U1.6 (D7): now also R8.2, SW8.1; no longer SW8.2
- net at R20.2, SW20.1: now also U4.14 (D3)
- net at R32.2, SW32.1: now also U5.6 (D7)
- net at R26.2, SW26.1: now also U5.12 (D1)
- net at U5.4 (D5): now also R30.2, SW30.1; no longer SW30.2
- net at U5.5 (D6): now also R31.2, SW31.1; no longer SW31.2
- net at U5.7 (~{Q7}): now also U3.21 (GPIO16)
- net at U5.9 (Q7): no longer U3.21 (GPIO16)
- net at R22.2, SW22.1: now also U4.4 (D5)
Other:
- moved on the sheet: R1, R10, R11, R12, R13, R14, R15, R16, R17, R18, R19, R2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
